Commit message: docs: add ROS2 internship portfolio README

File: assets/cell035/urdf/mini_4wd_robot_with_laser_drive_cell035.urdf (robot description, URDF)
Before this commit: robot mini_4wd_robot, 8 links, 7 joints
Links:
- link base_link: geometry collision mesh filename=package://wheeltec_robot_urdf/wheeltec_robot_urdf/meshes/mi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; visual mesh filename=package://wheeltec_robot_urdf/wheeltec_robot_urdf/meshes/mi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
- link camera_link: geometry collision mesh filename=package://wheeltec_robot_urdf/wheeltec_robot_urdf/meshes/mi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; visual mesh filename=package://wheeltec_robot_urdf/wheeltec_robot_urdf/meshes/mi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
- link controller_link: geometry collision mesh filename=package://wheeltec_robot_urdf/wheeltec_robot_urdf/meshes/mi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; visual mesh filename=package://wheeltec_robot_urdf/wheeltec_robot_urdf/meshes/mi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
- link laser_link: geometry collision mesh filename=package://wheeltec_robot_urdf/wheeltec_robot_urdf/meshes/mi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; visual mesh filename=package://wheeltec_robot_urdf/wheeltec_robot_urdf/meshes/mi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
- link lb_wheel_link: geometry collision mesh filename=package://wheeltec_robot_urdf/wheeltec_robot_urdf/meshes/mi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; visual mesh filename=package://wheeltec_robot_urdf/wheeltec_robot_urdf/meshes/mi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
- link lf_wheel_link: geometry collision mesh filename=package://wheeltec_robot_urdf/wheeltec_robot_urdf/meshes/mi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; visual mesh filename=package://wheeltec_robot_urdf/wheeltec_robot_urdf/meshes/mi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
- link rb_wheel_link: geometry collision mesh filename=package://wheeltec_robot_urdf/wheeltec_robot_urdf/meshes/mi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; visual mesh filename=package://wheeltec_robot_urdf/wheeltec_robot_urdf/meshes/mi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
- link rf_wheel_link: geometry collision mesh filename=package://wheeltec_robot_urdf/wheeltec_robot_urdf/meshes/mi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; visual mesh filename=package://wheeltec_robot_urdf/wheeltec_robot_urdf/meshes/mi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

File: assets/cell035/urdf/mini_4wd_robot_with_laser_drive_cell035_lidar360.urdf (robot description, URDF)
Before this commit: robot mini_4wd_robot, 8 links, 7 joints
Links:
- link base_link: geometry collision mesh filename=package://wheeltec_robot_urdf/wheeltec_robot_urdf/meshes/mi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; visual mesh filename=package://wheeltec_robot_urdf/wheeltec_robot_urdf/meshes/mi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
- link camera_link: geometry collision mesh filename=package://wheeltec_robot_urdf/wheeltec_robot_urdf/meshes/mi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; visual mesh filename=package://wheeltec_robot_urdf/wheeltec_robot_urdf/meshes/mi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
- link controller_link: geometry collision mesh filename=package://wheeltec_robot_urdf/wheeltec_robot_urdf/meshes/mi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; visual mesh filename=package://wheeltec_robot_urdf/wheeltec_robot_urdf/meshes/mi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
- link laser_link: geometry collision mesh filename=package://wheeltec_robot_urdf/wheeltec_robot_urdf/meshes/mi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; visual mesh filename=package://wheeltec_robot_urdf/wheeltec_robot_urdf/meshes/mi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
- link lb_wheel_link: geometry collision mesh filename=package://wheeltec_robot_urdf/wheeltec_robot_urdf/meshes/mi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; visual mesh filename=package://wheeltec_robot_urdf/wheeltec_robot_urdf/meshes/mi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
- link lf_wheel_link: geometry collision mesh filename=package://wheeltec_robot_urdf/wheeltec_robot_urdf/meshes/mi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; visual mesh filename=package://wheeltec_robot_urdf/wheeltec_robot_urdf/meshes/mi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
- link rb_wheel_link: geometry collision mesh filename=package://wheeltec_robot_urdf/wheeltec_robot_urdf/meshes/mi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; visual mesh filename=package://wheeltec_robot_urdf/wheeltec_robot_urdf/meshes/mi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
- link rf_wheel_link: geometry collision mesh filename=package://wheeltec_robot_urdf/wheeltec_robot_urdf/meshes/mi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; visual mesh filename=package://wheeltec_robot_urdf/wheeltec_robot_urdf/meshes/mi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
